File: MC_CP/Exquisite Blorr.brd (EAGLE design)
At the start: 298.3 x 227.1 mm, 9 parts, among them U7 ARDUINO-UNO-R3-SHIELD, U8 LCD-16X2JHD-162A, U9 ARDUINO-UNO-R3-SHIELD

Commit message: submitt
Parts:
- moved RPOT4 31.9 mm to (268.5, 188.1)
- moved SERVO3 0.30 mm to (291.5, 93.1)
Other:
- board size 298.3 x 227.1 mm -> 298.5 x 207.2 mm
Changed lines of the file:
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@@
 <board>
 <plain>
-<wire x1="0" y1="0" x2="298.283030487728" y2="0" width="0" layer="20"/>
-<wire x1="298.283030487728" y1="0" x2="298.283030487728" y2="227.06858226446423" width="0" layer="20"/>
-<wire x1="298.283030487728" y1="227.06858226446423" x2="0" y2="227.06858226446423" width="0" layer="20"/>
-<wire x1="0" y1="227.06858226446423" x2="0" y2="0" width="0" layer="20"/>
+<wire x1="0" y1="0" x2="298.49195217656325" y2="0" width="0" layer="20"/>
+<wire x1="298.49195217656325" y1="0" x2="298.49195217656325" y2="207.2307465436499" width="0" layer="20"/>
+<wire x1="298.49195217656325" y1="207.2307465436499" x2="0" y2="207.2307465436499" width="0" layer="20"/>
+<wire x1="0" y1="207.2307465436499" x2="0" y2="0" width="0" layer="20"/>
 </plain>
 <attributes/>
@@
 <element name="U8" library="Tinkercad" package="JHD-162A" package3d_urn="urn:adsk.eagle:package:32395061/2" value="LCD-16X2JHD-162A" x="239.2635" y="183.1477" smashed="yes"/>
 <element name="U9" library="Tinkercad" package="ARDUINO-UNO-R3-SHIELD" package3d_urn="urn:adsk.eagle:package:32092383/4" value="ARDUINO-UNO-R3-SHIELD" x="90.3686" y="47.885" smashed="yes"/>
-<element name="SERVO3" library="Tinkercad" package="SG90" package3d_urn="urn:adsk.eagle:package:32659983/2" value="SERVOSG90" x="291.298" y="92.9142" rot="R-270" smashed="yes"/>
-<element name="RPOT4" library="Tinkercad" package="HA-06-SM065" package3d_urn="urn:adsk.eagle:package:31496083/2" value="250k" x="268.029" y="220.0201" smashed="yes"/>
+<element name="SERVO3" library="Tinkercad" package="SG90" package3d_urn="urn:adsk.eagle:package:32659983/2" value="SERVOSG90" x="291.507" y="93.1231" rot="R-270" smashed="yes"/>
+<element name="RPOT4" library="Tinkercad" package="HA-06-SM065" package3d_urn="urn:adsk.eagle:package:31496083/2" value="250k" x="268.4735" y="188.1007" smashed="yes"/>
 <element name="R6" library="Tinkercad" package="RESAD1016W63L850D250B" package3d_urn="urn:adsk.eagle:package:31513020/2" value="330" x="8.2025" y="133.1896" rot="R90" smashed="yes"/>
 <element name="D3" library="Tinkercad" package="LEDRD254W60D565H860B" package3d_urn="urn:adsk.eagle:package:16378508/2" value="RED" x="9.4725" y="138.2696" rot="R180" smashed="yes">
@@
 <contactref element="U7" pad="GND@1"/>
 <contactref element="U7" pad="GND@2"/>
-<contactref element="RPOT4" pad="1"/>
 <contactref element="SERVO3" pad="1"/>
 <contactref element="U9" pad="GND@0"/>
@@
 <contactref element="U8" pad="5"/>
 <contactref element="R5" pad="2"/>
+<contactref element="RPOT4" pad="1"/>
 <contactref element="R6" pad="1"/>
 <wire x1="114.4986" y1="50.425" x2="114.4986" y2="52.965" width="0" layer="19" extent="1-1"/>
@@
 <wire x1="220.2135" y1="183.1477" x2="230.3735" y2="183.1477" width="0" layer="19" extent="1-1"/>
 <wire x1="230.3735" y1="183.1477" x2="258.3135" y2="203.3407" width="0" layer="19" extent="1-1"/>
-<wire x1="265.489" y1="217.4801" x2="258.3135" y2="203.3407" width="0" layer="19" extent="1-1"/>
-<wire x1="291.298" y1="90.3742" x2="230.3735" y2="183.1477" width="0" layer="19" extent="1-1"/>
+<wire x1="258.3135" y1="203.3407" x2="265.9335" y2="185.5607" width="0" layer="19" extent="1-1"/>
+<wire x1="291.507" y1="90.5831" x2="265.9335" y2="185.5607" width="0" layer="19" extent="1-1"/>
 </signal>
 <signal name="U8_LED-">
@@
 <signal name="U7_5V">
 <contactref element="U7" pad="5V"/>
-<contactref element="RPOT4" pad="3"/>
 <contactref element="SERVO3" pad="2"/>
 <contactref element="U9" pad="5V"/>
 <contactref element="U8" pad="2"/>
 <contactref element="U8" pad="15"/>
+<contactref element="RPOT4" pad="3"/>
+<wire x1="255.7735" y1="183.1477" x2="271.0135" y2="185.5607" width="0" layer="19" extent="1-1"/>
 <wire x1="222.7535" y1="183.1477" x2="255.7735" y2="183.1477" width="0" layer="19" extent="1-1"/>
-<wire x1="270.569" y1="217.4801" x2="255.7735" y2="183.1477" width="0" layer="19" extent="1-1"/>
-<wire x1="291.298" y1="92.9142" x2="255.7735" y2="183.1477" width="0" layer="19" extent="1-1"/>
+<wire x1="291.507" y1="93.1231" x2="271.0135" y2="185.5607" width="0" layer="19" extent="1-1"/>
 <wire x1="109.211" y1="140.8595" x2="222.7535" y2="183.1477" width="0" layer="19" extent="1-1"/>
 <wire x1="109.211" y1="140.8595" x2="114.4986" y2="47.885" width="0" layer="19" extent="1-1"/>
@@
 </signal>
 <signal name="U8_VO">
+<contactref element="U8" pad="3"/>
 <contactref element="RPOT4" pad="2"/>
-<contactref element="U8" pad="3"/>
-<wire x1="268.029" y1="222.5601" x2="225.2935" y2="183.1477" width="0" layer="19" extent="1-1"/>
+<wire x1="225.2935" y1="183.1477" x2="268.4735" y2="190.6407" width="0" layer="19" extent="1-1"/>
 </signal>
 <signal name="U9_D9">
 <contactref element="SERVO3" pad="3"/>
 <contactref element="U9" pad="D9"/>
-<wire x1="291.298" y1="95.4542" x2="66.2386" y2="49.155" width="0" layer="19" extent="1-1"/>
+<wire x1="291.507" y1="95.6631" x2="66.2386" y2="49.155" width="0" layer="19" extent="1-1"/>
 </signal>
 <signal name="D3_C">
